File: kicad-project-template/kicad-project-template.kicad_sch (KiCad schematic)
At the start: 0 parts

Commit message: Updated logos and sheet naming to everyday dev
Other:
- note removed: "great lakes dev"
- company: great lakes dev -> everyday dev

Commit message: Added manufacturer to bom output and updated MFP to MPN to follow other standards
Parts:
- added R1: 10k, Resistor_SMD:R_0402_1005Metric, symbol Device:R_Small_US
Connections:
- new net GND: R1.2
- new net VCC: R1.1
Changed lines of the file:
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@@
     (comment 1 "License: CC-BY-SA")
+  )
+  (wire (pts (xy 134.62 104.14) (xy 134.62 106.68))
+    (stroke (width 0) (type default))
+  )
+  (wire (pts (xy 134.62 96.52) (xy 134.62 99.06))
+    (stroke (width 0) (type default))
   )
   (image (at 193.04 170.18) (scale 0.303569)
@@
     )
   )
+  (symbol (lib_id "Device:R_Small_US") (at 134.62 101.6 0) (unit 1)
+    (in_bom yes) (on_board yes) (dnp no) (fields_autoplaced)
+    (property "Reference" "R1" (at 137.16 100.33 0)
+      (effects (font (size 1.27 1.27)) (justify left))
+    )
+    (property "Value" "10k" (at 137.16 102.87 0)
+      (effects (font (size 1.27 1.27)) (justify left))
+    )
+    (property "Footprint" "Resistor_SMD:R_0402_1005Metric" (at 134.62 101.6 0)
+      (effects (font (size 1.27 1.27)) hide)
+    )
+    (property "Datasheet" "~" (at 134.62 101.6 0)
+      (effects (font (size 1.27 1.27)) hide)
+    )
+    (property "MPN" "~" (at 134.62 101.6 0)
+      (effects (font (size 1.27 1.27)) hide)
+    )
+    (property "Manufacturer" "~" (at 134.62 101.6 0)
+      (effects (font (size 1.27 1.27)) hide)
+    )
+    (pin "1")
+    (pin "2")
+    (instances
+      (project "kicad-project-template"
+        (path "/bd7ed9f8-b5b4-423c-a38d-d164cc860cc9"
+          (reference "R1") (unit 1)
+        )
+      )
+    )
+  )
+  (symbol (lib_id "power:VCC") (at 134.62 96.52 0) (unit 1)
+    (in_bom yes) (on_board yes) (dnp no) (fields_autoplaced)
+    (property "Reference" "#PWR02" (at 134.62 100.33 0)
+      (effects (font (size 1.27 1.27)) hide)
+    )
+    (property "Value" "VCC" (at 134.62 91.44 0)
+      (effects (font (size 1.27 1.27)))
+    )
+    (property "Footprint" "" (at 134.62 96.52 0)
+      (effects (font (size 1.27 1.27)) hide)
+    )
+    (property "Datasheet" "" (at 134.62 96.52 0)
+      (effects (font (size 1.27 1.27)) hide)
+    )
+    (pin "1")
+    (instances
+      (project "kicad-project-template"
+        (path "/bd7ed9f8-b5b4-423c-a38d-d164cc860cc9"
+          (reference "#PWR02") (unit 1)
+        )
+      )
+    )
+  )
+  (symbol (lib_id "power:GND") (at 134.62 106.68 0) (unit 1)
+    (in_bom yes) (on_board yes) (dnp no) (fields_autoplaced)
+    (property "Reference" "#PWR01" (at 134.62 113.03 0)
+      (effects (font (size 1.27 1.27)) hide)
+    )
+    (property "Value" "GND" (at 134.62 111.76 0)
+      (effects (font (size 1.27 1.27)))
+    )
+    (property "Footprint" "" (at 134.62 106.68 0)
+      (effects (font (size 1.27 1.27)) hide)
+    )
+    (property "Datasheet" "" (at 134.62 106.68 0)
+      (effects (font (size 1.27 1.27)) hide)
+    )
+    (pin "1")
+    (instances
+      (project "kicad-project-template"
+        (path "/bd7ed9f8-b5b4-423c-a38d-d164cc860cc9"
+          (reference "#PWR01") (unit 1)
+        )
+      )
+    )
+  )
